Commit message: added new camera, correct positioning

File: urdf/butler.xacro (robot description, xacro)
@@ -1,4 +1,6 @@
 <?xml version="1.0" ?>
 <robot name="butler" xmlns:xacro="http://www.ros.org/wiki/xacro">
+<xacro:property name="cameraSize" value="0.05"/>
+<xacro:property name="cameraMass" value="0.1"/>
 <xacro:include filename="$(find butler_description)/urdf/materials.xacro" />
 <xacro:include filename="$(find butler_description)/urdf/butler.trans" />
@@ -1378,3 +1380,30 @@
   <child link="Caster_22455T16_c_rod_v1_1"/>
 </joint>
+<link name="camera">
+    <collision>
+      <origin xyz="0 0 0" rpy="0 0 0"/>
+      <geometry>
+        <box size="${cameraSize} ${cameraSize} ${cameraSize}"/>
+      </geometry>
+    </collision>
+    <visual>
+      <origin xyz="0 0 0" rpy="0 0 0"/>
+      <geometry>
+        <box size="${cameraSize} ${cameraSize} ${cameraSize}"/>
+      </geometry>
+      <material name="green"/>
+    </visual>
+    <inertial>
+      <mass value="${cameraMass}" />
+      <origin xyz="0 0 0" rpy="0 0 0"/>
+      <box_inertia m="${cameraMass}" x="${cameraSize}" y="${cameraSize}" z="${cameraSize}" />
+      <inertia ixx="1e-6" ixy="0" ixz="0" iyy="1e-6" iyz="0" izz="1e-6" />
+    </inertial>
+  </link>
+  <joint name="camera_joint" type="fixed">
+    <axis xyz="0 1 0" />
+    <origin xyz="-0.4 0.0005 0.04" rpy="0 0 1.57"/>
+    <parent link="Upper_Plate_v95__2__1"/>
+    <child link="camera"/>
+  </joint>
 </robot>

Commit message: added lasers second plate

File: urdf/butler.xacro (robot description, xacro)
@@ -1307,4 +1307,5 @@
 </joint>
 <joint name="Rigid44" type="fixed">
+  <axis xyz="0 1 0" />
   <origin rpy="0 0 0" xyz="-0.117824 -0.005002 0.00635"/>
   <parent link="Upper_Plate_v95__1__1"/>
@@ -1345,5 +1346,5 @@
   <parent link="butler_motor_v1_1"/>
   <child link="butler_tire_v1_1"/>
-  <axis xyz="1.0 0.0 -0.0"/>
+  <axis xyz="-1.0 0.0 0.0"/>
 </joint>
 <joint name="Rigid53" type="fixed">
@@ -1381,24 +1382,24 @@
 </joint>
 <link name="camera">
-    <collision>
-      <origin xyz="0 0 0" rpy="0 0 0"/>
-      <geometry>
-        <box size="${cameraSize} ${cameraSize} ${cameraSize}"/>
-      </geometry>
-    </collision>
-    <visual>
-      <origin xyz="0 0 0" rpy="0 0 0"/>
-      <geometry>
-        <box size="${cameraSize} ${cameraSize} ${cameraSize}"/>
-      </geometry>
-      <material name="green"/>
-    </visual>
-    <inertial>
-      <mass value="${cameraMass}" />
-      <origin xyz="0 0 0" rpy="0 0 0"/>
-      <box_inertia m="${cameraMass}" x="${cameraSize}" y="${cameraSize}" z="${cameraSize}" />
-      <inertia ixx="1e-6" ixy="0" ixz="0" iyy="1e-6" iyz="0" izz="1e-6" />
-    </inertial>
-  </link>
+  <collision>
+    <origin xyz="0 0 0" rpy="0 0 0"/>
+    <geometry>
+      <box size="${cameraSize} ${cameraSize} ${cameraSize}"/>
+    </geometry>
+  </collision>
+  <visual>
+    <origin xyz="0 0 0" rpy="0 0 0"/>
+    <geometry>
+      <box size="${cameraSize} ${cameraSize} ${cameraSize}"/>
+    </geometry>
+    <material name="green"/>
+  </visual>
+  <inertial>
+    <mass value="${cameraMass}" />
+    <origin xyz="0 0 0" rpy="0 0 0"/>
+    <box_inertia m="${cameraMass}" x="${cameraSize}" y="${cameraSize}" z="${cameraSize}" />
+    <inertia ixx="1e-6" ixy="0" ixz="0" iyy="1e-6" iyz="0" izz="1e-6" />
+  </inertial>
+</link>
   <joint name="camera_joint" type="fixed">
     <axis xyz="0 1 0" />
@@ -1407,3 +1408,55 @@
     <child link="camera"/>
   </joint>
+  <joint name="laser_joint_tail" type="fixed">
+    <axis xyz="0 1 0" />
+    <origin rpy="0 0 -1.57" xyz="0.31 -0.72 0.04"/>
+    <parent link="Upper_Plate_v95_1"/>
+    <child link="laser_tail"/>
+  </joint>
+  <!-- Hokuyo Laser -->
+  <link name="laser_tail">
+    <collision>
+      <origin xyz="0 0 0" rpy="0 0 0"/>
+      <geometry>
+    <box size="0.1 0.1 0.1"/>
+      </geometry>
+    </collision>
+    <visual>
+      <origin xyz="0 0 0" rpy="0 0 0"/>
+      <geometry>
+        <mesh filename="package://butler_description/meshes/laser_hokuyo.dae"/>
+      </geometry>
+    </visual>
+    <inertial>
+      <mass value="1e-5" />
+      <origin xyz="0 0 0" rpy="0 0 0"/>
+      <inertia ixx="1e-6" ixy="0" ixz="0" iyy="1e-6" iyz="0" izz="1e-6" />
+    </inertial>
+  </link>
+  <joint name="laser_joint_head" type="fixed">
+    <axis xyz="0 1 0" />
+  <origin rpy="0 0 1.57" xyz="0.31 0 0.04"/>
+  <parent link="Upper_Plate_v95_1"/>
+  <child link="laser_head"/>
+  </joint>
+  <!-- Hokuyo Laser -->
+  <link name="laser_head">
+  <collision>
+    <origin xyz="0 0 0" rpy="0 0 0"/>
+    <geometry>
+  <box size="0.1 0.1 0.1"/>
+    </geometry>
+  </collision>
+  <visual>
+    <origin xyz="0 0 0" rpy="0 0 0"/>
+    <geometry>
+      <mesh filename="package://butler_description/meshes/laser_hokuyo.dae"/>
+    </geometry>
+  </visual>
+  <inertial>
+    <mass value="1e-5" />
+    <origin xyz="0 0 0" rpy="0 0 0"/>
+    <inertia ixx="1e-6" ixy="0" ixz="0" iyy="1e-6" iyz="0" izz="1e-6" />
+  </inertial>
+  </link>
 </robot>

Commit message: added lasers on second plate

File: urdf/butler.xacro (robot description, xacro)
@@ -1382,24 +1382,24 @@
 </joint>
 <link name="camera">
-  <collision>
-    <origin xyz="0 0 0" rpy="0 0 0"/>
-    <geometry>
-      <box size="${cameraSize} ${cameraSize} ${cameraSize}"/>
-    </geometry>
-  </collision>
-  <visual>
-    <origin xyz="0 0 0" rpy="0 0 0"/>
-    <geometry>
-      <box size="${cameraSize} ${cameraSize} ${cameraSize}"/>
-    </geometry>
-    <material name="green"/>
-  </visual>
-  <inertial>
-    <mass value="${cameraMass}" />
-    <origin xyz="0 0 0" rpy="0 0 0"/>
-    <box_inertia m="${cameraMass}" x="${cameraSize}" y="${cameraSize}" z="${cameraSize}" />
-    <inertia ixx="1e-6" ixy="0" ixz="0" iyy="1e-6" iyz="0" izz="1e-6" />
-  </inertial>
-</link>
+    <collision>
+      <origin xyz="0 0 0" rpy="0 0 0"/>
+      <geometry>
+        <box size="${cameraSize} ${cameraSize} ${cameraSize}"/>
+      </geometry>
+    </collision>
+    <visual>
+      <origin xyz="0 0 0" rpy="0 0 0"/>
+      <geometry>
+        <box size="${cameraSize} ${cameraSize} ${cameraSize}"/>
+      </geometry>
+      <material name="green"/>
+    </visual>
+    <inertial>
+      <mass value="${cameraMass}" />
+      <origin xyz="0 0 0" rpy="0 0 0"/>
+      <box_inertia m="${cameraMass}" x="${cameraSize}" y="${cameraSize}" z="${cameraSize}" />
+      <inertia ixx="1e-6" ixy="0" ixz="0" iyy="1e-6" iyz="0" izz="1e-6" />
+    </inertial>
+  </link>
   <joint name="camera_joint" type="fixed">
     <axis xyz="0 1 0" />

Commit message: fixed light fixtures in model

File: urdf/butler.xacro (robot description, xacro)
@@ -466,44 +466,4 @@
   </collision>
 </link>
-<link name="GAU-LP-3L-UVC-T8-V1_3ft_Light_v5__1__1">
-  <inertial>
-    <origin rpy="0 0 0" xyz="0.030434930745823596 1.8742240127933574e-07 0.44743182523617936"/>
-    <mass value="2.6048863345120696"/>
-    <inertia ixx="0.199966" ixy="-0.0" ixz="0.001051" iyy="0.20026" iyz="0.0" izz="0.002331"/>
-  </inertial>
-  <visual>
-    <origin rpy="0 0 0" xyz="-0.34835 0.121336 -0.349551"/>
-    <geometry>
-      <mesh filename="package://butler_description/meshes/GAU-LP-3L-UVC-T8-V1_3ft_Light_v5__1__1.stl" scale="0.001 0.001 0.001"/>
-    </geometry>
-    <material name="silver"/>
-  </visual>
-  <collision>
-    <origin rpy="0 0 0" xyz="-0.34835 0.121336 -0.349551"/>
-    <geometry>
-      <mesh filename="package://butler_description/meshes/GAU-LP-3L-UVC-T8-V1_3ft_Light_v5__1__1.stl" scale="0.001 0.001 0.001"/>
-    </geometry>
-  </collision>
-</link>
-<link name="GAU-LP-3L-UVC-T8-V1_3ft_Light_v5_1">
-  <inertial>
-    <origin rpy="0 0 0" xyz="-0.030434352859068814 1.8742239775437763e-07 0.4474318252361786"/>
-    <mass value="2.6048863345120696"/>
-    <inertia ixx="0.199966" ixy="-0.0" ixz="-0.001051" iyy="0.20026" iyz="-0.0" izz="0.002331"/>
-  </inertial>
-  <visual>
-    <origin rpy="0 0 0" xyz="0.358866 0.121336 -0.349551"/>
-    <geometry>
-      <mesh filename="package://butler_description/meshes/GAU-LP-3L-UVC-T8-V1_3ft_Light_v5_1.stl" scale="0.001 0.001 0.001"/>
-    </geometry>
-    <material name="silver"/>
-  </visual>
-  <collision>
-    <origin rpy="0 0 0" xyz="0.358866 0.121336 -0.349551"/>
-    <geometry>
-      <mesh filename="package://butler_description/meshes/GAU-LP-3L-UVC-T8-V1_3ft_Light_v5_1.stl" scale="0.001 0.001 0.001"/>
-    </geometry>
-  </collision>
-</link>
 <link name="Upper_Plate_v95__1__1">
   <inertial>
@@ -666,24 +626,4 @@
   </collision>
 </link>
-<link name="GAU-LP-3L-UVC-T8-V1_2ft_v5_1">
-  <inertial>
-    <origin rpy="0 0 0" xyz="0.03043493074582443 1.8742237754831859e-07 0.34452233580782665"/>
-    <mass value="2.005762477574293"/>
-    <inertia ixx="0.091611" ixy="-0.0" ixz="0.000623" iyy="0.091837" iyz="0.0" izz="0.001795"/>
-  </inertial>
-  <visual>
-    <origin rpy="0 0 0" xyz="-0.34835 0.121336 -1.442672"/>
-    <geometry>
-      <mesh filename="package://butler_description/meshes/GAU-LP-3L-UVC-T8-V1_2ft_v5_1.stl" scale="0.001 0.001 0.001"/>
-    </geometry>
-    <material name="silver"/>
-  </visual>
-  <collision>
-    <origin rpy="0 0 0" xyz="-0.34835 0.121336 -1.442672"/>
-    <geometry>
-      <mesh filename="package://butler_description/meshes/GAU-LP-3L-UVC-T8-V1_2ft_v5_1.stl" scale="0.001 0.001 0.001"/>
-    </geometry>
-  </collision>
-</link>
 <link name="gusset_4_1">
   <inertial>
@@ -726,24 +666,4 @@
   </collision>
 </link>
-<link name="GAU-LP-3L-UVC-T8-V1_2ft_v5__1__1">
-  <inertial>
-    <origin rpy="0 0 0" xyz="-0.03043435285906787 1.8742237396784933e-07 0.3445223358078262"/>
-    <mass value="2.005762477574293"/>
-    <inertia ixx="0.091611" ixy="-0.0" ixz="-0.000623" iyy="0.091837" iyz="-0.0" izz="0.001795"/>
-  </inertial>
-  <visual>
-    <origin rpy="0 0 0" xyz="0.358866 0.121336 -1.442672"/>
-    <geometry>
-      <mesh filename="package://butler_description/meshes/GAU-LP-3L-UVC-T8-V1_2ft_v5__1__1.stl" scale="0.001 0.001 0.001"/>
-    </geometry>
-    <material name="silver"/>
-  </visual>
-  <collision>
-    <origin rpy="0 0 0" xyz="0.358866 0.121336 -1.442672"/>
-    <geometry>
-      <mesh filename="package://butler_description/meshes/GAU-LP-3L-UVC-T8-V1_2ft_v5__1__1.stl" scale="0.001 0.001 0.001"/>
-    </geometry>
-  </collision>
-</link>
 <link name="Upper_Plate_v95__2__1">
   <inertial>
@@ -1103,4 +1023,84 @@
     <geometry>
       <mesh filename="package://butler_description/meshes/Caster_22455T16_c_rod_v1_1.stl" scale="0.001 0.001 0.001"/>
+    </geometry>
+  </collision>
+</link>
+<link name="3ft_light_fixture_v1__1__1">
+  <inertial>
+    <origin rpy="0 0 0" xyz="-0.5309020692540334 -0.07337799454852041 0.8260446180764844"/>
+    <mass value="2.60488633452387"/>
+    <inertia ixx="0.199966" ixy="0.0" ixz="-0.001051" iyy="0.20026" iyz="0.0" izz="0.002331"/>
+  </inertial>
+  <visual>
+    <origin rpy="0 0 0" xyz="-0.909687 0.025533 0.0"/>
+    <geometry>
+      <mesh filename="package://butler_description/meshes/3ft_light_fixture_v1__1__1.stl" scale="0.001 0.001 0.001"/>
+    </geometry>
+    <material name="silver"/>
+  </visual>
+  <collision>
+    <origin rpy="0 0 0" xyz="-0.909687 0.025533 0.0"/>
+    <geometry>
+      <mesh filename="package://butler_description/meshes/3ft_light_fixture_v1__1__1.stl" scale="0.001 0.001 0.001"/>
+    </geometry>
+  </collision>
+</link>
+<link name="3ft_light_fixture_v1_1">
+  <inertial>
+    <origin rpy="0 0 0" xyz="-1.2989873528592129 -0.1244439945483815 0.8260446180764848"/>
+    <mass value="2.60488633452387"/>
+    <inertia ixx="0.199966" ixy="0.0" ixz="0.001051" iyy="0.20026" iyz="0.0" izz="0.002331"/>
+  </inertial>
+  <visual>
+    <origin rpy="0 0 0" xyz="-0.909687 -0.025533 0.0"/>
+    <geometry>
+      <mesh filename="package://butler_description/meshes/3ft_light_fixture_v1_1.stl" scale="0.001 0.001 0.001"/>
+    </geometry>
+    <material name="silver"/>
+  </visual>
+  <collision>
+    <origin rpy="0 0 0" xyz="-0.909687 -0.025533 0.0"/>
+    <geometry>
+      <mesh filename="package://butler_description/meshes/3ft_light_fixture_v1_1.stl" scale="0.001 0.001 0.001"/>
+    </geometry>
+  </collision>
+</link>
+<link name="2ft_light_fixture_v1__1__1">
+  <inertial>
+    <origin rpy="0 0 0" xyz="-0.5279810692540323 -0.07337799454854385 1.809571916294862"/>
+    <mass value="2.0057624775833927"/>
+    <inertia ixx="0.091611" ixy="0.0" ixz="-0.000623" iyy="0.091837" iyz="0.0" izz="0.001795"/>
+  </inertial>
+  <visual>
+    <origin rpy="0 0 0" xyz="-0.906766 0.025533 0.0"/>
+    <geometry>
+      <mesh filename="package://butler_description/meshes/2ft_light_fixture_v1__1__1.stl" scale="0.001 0.001 0.001"/>
+    </geometry>
+    <material name="silver"/>
+  </visual>
+  <collision>
+    <origin rpy="0 0 0" xyz="-0.906766 0.025533 0.0"/>
+    <geometry>
+      <mesh filename="package://butler_description/meshes/2ft_light_fixture_v1__1__1.stl" scale="0.001 0.001 0.001"/>
+    </geometry>
+  </collision>
+</link>
+<link name="2ft_light_fixture_v1_1">
+  <inertial>
+    <origin rpy="0 0 0" xyz="-1.2960663528592116 -0.12444399454840412 1.8095719162948618"/>
+    <mass value="2.0057624775833927"/>
+    <inertia ixx="0.091611" ixy="0.0" ixz="0.000623" iyy="0.091837" iyz="-0.0" izz="0.001795"/>
+  </inertial>
+  <visual>
+    <origin rpy="0 0 0" xyz="-0.906766 -0.025533 0.0"/>
+    <geometry>
+      <mesh filename="package://butler_description/meshes/2ft_light_fixture_v1_1.stl" scale="0.001 0.001 0.001"/>
+    </geometry>
+    <material name="silver"/>
+  </visual>
+  <collision>
+    <origin rpy="0 0 0" xyz="-0.906766 -0.025533 0.0"/>
+    <geometry>
+      <mesh filename="package://butler_description/meshes/2ft_light_fixture_v1_1.stl" scale="0.001 0.001 0.001"/>
     </geometry>
   </collision>
@@ -1216,14 +1216,4 @@
   <child link="25-2525-BLACK-FB-3ft_v4_1"/>
 </joint>
-<joint name="Rigid26" type="fixed">
-  <origin rpy="0 0 0" xyz="0.0125 -0.00432 0.0"/>
-  <parent link="25-2525-BLACK-FB-3ft_v4_1"/>
-  <child link="GAU-LP-3L-UVC-T8-V1_3ft_Light_v5__1__1"/>
-</joint>
-<joint name="Rigid27" type="fixed">
-  <origin rpy="0 0 0" xyz="-0.0125 -0.00432 0.0"/>
-  <parent link="25-2525-BLACK-FB-3ft_v4__1__1"/>
-  <child link="GAU-LP-3L-UVC-T8-V1_3ft_Light_v5_1"/>
-</joint>
 <joint name="Rigid28" type="fixed">
   <origin rpy="0 0 0" xyz="0.0 0.0 1.086771"/>
@@ -1266,9 +1256,4 @@
   <child link="25-2525-BLACK-FB_v5_1"/>
 </joint>
-<joint name="Rigid36" type="fixed">
-  <origin rpy="0 0 0" xyz="0.0125 -0.00432 0.0"/>
-  <parent link="25-2525-BLACK-FB_v5_1"/>
-  <child link="GAU-LP-3L-UVC-T8-V1_2ft_v5_1"/>
-</joint>
 <joint name="Rigid37" type="fixed">
   <origin rpy="0 0 0" xyz="-0.459869 0.297649 0.00635"/>
@@ -1280,9 +1265,4 @@
   <parent link="Upper_Plate_v95__1__1"/>
   <child link="25-2525-BLACK-FB_v5__1__1"/>
-</joint>
-<joint name="Rigid39" type="fixed">
-  <origin rpy="0 0 0" xyz="-0.0125 -0.00432 0.0"/>
-  <parent link="25-2525-BLACK-FB_v5__1__1"/>
-  <child link="GAU-LP-3L-UVC-T8-V1_2ft_v5__1__1"/>
 </joint>
 <joint name="Rigid40" type="fixed">
@@ -1380,4 +1360,24 @@
   <parent link="Caster_22455T16_c_holder_v1_1"/>
   <child link="Caster_22455T16_c_rod_v1_1"/>
+</joint>
+<joint name="Rigid60" type="fixed">
+  <origin rpy="0 0 0" xyz="0.573837 0.091483 -0.349551"/>
+  <parent link="25-2525-BLACK-FB-3ft_v4_1"/>
+  <child link="3ft_light_fixture_v1__1__1"/>
+</joint>
+<joint name="Rigid61" type="fixed">
+  <origin rpy="0 0 0" xyz="1.256053 0.142549 -0.349551"/>
+  <parent link="25-2525-BLACK-FB-3ft_v4__1__1"/>
+  <child link="3ft_light_fixture_v1_1"/>
+</joint>
+<joint name="Rigid62" type="fixed">
+  <origin rpy="0 0 0" xyz="0.570916 0.091483 -1.442672"/>
+  <parent link="25-2525-BLACK-FB_v5_1"/>
+  <child link="2ft_light_fixture_v1__1__1"/>
+</joint>
+<joint name="Rigid63" type="fixed">
+  <origin rpy="0 0 0" xyz="1.253132 0.142549 -1.442672"/>
+  <parent link="25-2525-BLACK-FB_v5__1__1"/>
+  <child link="2ft_light_fixture_v1_1"/>
 </joint>
 <link name="camera">
