Commit message: added hokuyo, changed laser to ray

File: urdf/coach_butler_robot.urdf (robot description, URDF)
Before this commit: robot coach_butler_robot, 9 links, 8 joints
Links:
- link front_laser: geometry collision mesh filename=package://butler_description/meshes/hokuyo.dae; visual mesh filename=package://butler_description/meshes/hokuyo.dae

Commit message: incorporated covid killer robot urdf

File: urdf/coach_butler_robot.urdf (robot description, URDF)
Before this commit: robot coach_butler_robot, 9 links, 8 joints
Links:
- removed link left_caster
- removed link left_swivel
- removed link rear_laser
- removed link right_caster
- removed link right_swivel
- added link back_left_caster, mass 0.442987770505456; collision mesh filename=package://butler_description/meshes/back_left_caster.STL; visual mesh filename=package://butler_description/meshes/back_left_caster.STL
- added link back_left_swivel, mass 1.59345861527837; collision mesh filename=package://butler_description/meshes/back_left_swivel.STL; visual mesh filename=package://butler_description/meshes/back_left_swivel.STL
- added link back_right_caster, mass 0.44299; collision mesh filename=package://butler_description/meshes/back_right_caster.STL; visual mesh filename=package://butler_description/meshes/back_right_caster.STL
- added link back_right_swivel, mass 1.5935; collision mesh filename=package://butler_description/meshes/back_right_swivel.STL; visual mesh filename=package://butler_description/meshes/back_right_swivel.STL
- added link front_left_caster, mass 0.442987770505456; collision mesh filename=package://butler_description/meshes/front_left_caster.STL; visual mesh filename=package://butler_description/meshes/front_left_caster.STL
- added link front_left_swivel, mass 1.59345861527837; collision mesh filename=package://butler_description/meshes/front_left_swivel.STL; visual mesh filename=package://butler_description/meshes/front_left_swivel.STL
- added link front_right_caster, mass 0.44299; collision mesh filename=package://butler_description/meshes/front_right_caster.STL; visual mesh filename=package://butler_description/meshes/front_right_caster.STL
- added link front_right_swivel, mass 1.5935; collision mesh filename=package://butler_description/meshes/front_right_swivel.STL; visual mesh filename=package://butler_description/meshes/front_right_swivel.STL
- link base_link: mass 26.1616258468403 -> 32.099
- link front_laser: mass 1e-5 -> 0.36783; geometry collision mesh filename=package://butler_description/meshes/front_laser.STL; visual mesh filename=package://butler_description/meshes/front_laser.STL
- link left_wheel: mass 0.844079114777031 -> 0.84407911477703; geometry collision mesh filename=package://butler_description/meshes/left_wheel.STL; visual mesh filename=package://butler_description/meshes/left_wheel.STL
- link right_wheel: mass 0.844079114777032 -> 0.84408; geometry collision mesh filename=package://butler_description/meshes/right_wheel.STL; visual mesh filename=package://butler_description/meshes/right_wheel.STL
Joints:
- removed joint base_link_left_swivel
- removed joint base_link_rear_laser
- removed joint base_link_right_swivel
- removed joint left_swivel_left_caster
- removed joint right_swivel_right_caster
- added joint back_left_swivel_back_left_caster: type continuous, parent back_left_swivel, child back_left_caster, origin xyz=-0.04445 0 -0.071438 rpy=0 0 0, axis 0 -1 0
- added joint back_right_swivel_back_right_caster: type continuous, parent back_right_swivel, child back_right_caster, origin xyz=-0.04445 0 -0.071438 rpy=0 0 0, axis 0 -1 0
- added joint base_link_back_left_swivel: type continuous, parent base_link, child back_left_swivel, origin xyz=0.254 0.254 0.092538 rpy=0 0 -1.5708, axis 0 0 1
- added joint base_link_back_right_swivel: type continuous, parent base_link, child back_right_swivel, origin xyz=-0.254 0.254 0.092538 rpy=0 0 -1.5708, axis 0 0 1
- added joint base_link_front_left_swivel: type continuous, parent base_link, child front_left_swivel, origin xyz=0.254 -0.254 0.092538 rpy=0 0 -1.5708, axis 0 0 1
- added joint base_link_front_right_swivel: type continuous, parent base_link, child front_right_swivel, origin xyz=-0.254 -0.254 0.092538 rpy=0 0 -1.5708, axis 0 0 1
- added joint front_left_swivel_front_left_caster: type continuous, parent front_left_swivel, child front_left_caster, origin xyz=-0.04445 0 -0.071438 rpy=0 0 0, axis 0 -1 0
- added joint front_right_swivel_front_right_caster: type continuous, parent front_right_swivel, child front_right_caster, origin xyz=-0.04445 0 -0.071438 rpy=0 0 0, axis 0 1 0
- joint base_link_front_laser: axis 0 0 1 -> 0 0 -1; origin xyz=0.26865 0 0.043175 rpy=0 0 0 -> xyz=0 -0.38239 0.15967 rpy=0 0 -1.5708
- joint base_link_left_wheel: axis 0 1 0 -> 0 -1 0; origin xyz=0.173356333637394 0.27870625 0.0487011859215695 rpy=0 0 0 -> xyz=0.28302 0 0.048701 rpy=0 0 -1.5708
- joint base_link_right_wheel: origin xyz=0.17336 -0.27871 0.048701 rpy=0 0 0 -> xyz=-0.28302 0 0.048701 rpy=0 0 -1.5708

Commit message: fixed urdf issue in gazebo, added front laser

File: urdf/coach_butler_robot.urdf (robot description, URDF)
Before this commit: robot coach_butler_robot, 12 links, 11 joints
Links:
- link left_wheel: geometry collision cylinder length=0.03175 radius=0.08; visual mesh filename=package://butler_description/meshes/left_wheel.STL
- link right_wheel: geometry collision cylinder length=0.03175 radius=0.08; visual mesh filename=package://butler_description/meshes/right_wheel.STL
Joints:
- joint base_link_left_wheel: axis 0 -1 0 -> 0 1 0

Commit message: added rear laser to urdf

File: urdf/coach_butler_robot.urdf (robot description, URDF)
Before this commit: robot coach_butler_robot, 12 links, 11 joints
Links:
- added link rear_laser, mass 0.36783; collision mesh filename=package://butler_description/meshes/rear_laser.STL; visual mesh filename=package://butler_description/meshes/rear_laser.STL
Joints:
- added joint base_link_rear_laser: type revolute, parent base_link, child rear_laser, origin xyz=0 0.38239 0.15967 rpy=0 0 1.5708, axis 0 0 -1, limit lower=0 upper=0 effort=0 velocity=0

Commit message: added front camera to urdf

File: urdf/coach_butler_robot.urdf (robot description, URDF)
Before this commit: robot coach_butler_robot, 13 links, 12 joints
Links:
- added link front_camera, mass 0.1; collision box size=0.05 0.05 0.05; visual box size=0.05 0.05 0.05
Joints:
- added joint base_link_front_camera: type fixed, parent base_link, child front_camera, origin xyz=0 -0.35239 1.32 rpy=0 0 -1.5708, axis 0 1 0

Commit message: incorportated coach's new urdf, fixed base_link orientation

File: urdf/coach_butler_robot.urdf (robot description, URDF)
Before this commit: robot coach_butler_robot, 14 links, 13 joints
Links:
- removed link front_camera
- removed link rear_laser
- link back_right_caster: mass 0.44299 -> 0.442987770505456
- link back_right_swivel: mass 1.5935 -> 1.59345861527837
- link base_link: mass 32.099 -> 44.766149285195
- link front_right_caster: mass 0.44299 -> 0.442987770505456
- link front_right_swivel: mass 1.5935 -> 1.59345861527837
- link left_wheel: mass 0.84407911477703 -> 0.844079114777031
- link right_wheel: mass 0.84408 -> 0.844079114777031
Joints:
- removed joint base_link_front_camera
- removed joint base_link_rear_laser
- joint back_left_swivel_back_left_caster: origin xyz=-0.04445 0 -0.071438 rpy=0 0 0 -> xyz=-0.04445 0 -0.0714375 rpy=0 0 0
- joint back_right_swivel_back_right_caster: origin xyz=-0.04445 0 -0.071438 rpy=0 0 0 -> xyz=-0.04445 0 -0.0714375 rpy=0 0 0
- joint base_link_back_left_swivel: origin xyz=0.254 0.254 0.092538 rpy=0 0 -1.5708 -> xyz=-0.254 0.254 0.0957125000000003 rpy=0 0 0
- joint base_link_back_right_swivel: origin xyz=-0.254 0.254 0.092538 rpy=0 0 -1.5708 -> xyz=-0.254 -0.254 0.095712 rpy=0 0 0
- joint base_link_front_laser: origin xyz=0 -0.38239 0.15967 rpy=0 0 -1.5708 -> xyz=0.38239 0 0.15967 rpy=0 0 0
- joint base_link_front_left_swivel: origin xyz=0.254 -0.254 0.092538 rpy=0 0 -1.5708 -> xyz=0.254 0.254 0.095713 rpy=0 0 0
- joint base_link_front_right_swivel: origin xyz=-0.254 -0.254 0.092538 rpy=0 0 -1.5708 -> xyz=0.254 -0.254 0.095712 rpy=0 0 0
- joint base_link_left_wheel: origin xyz=0.28302 0 0.048701 rpy=0 0 -1.5708 -> xyz=0 0.28302 0.051876 rpy=0 0 0
- joint base_link_right_wheel: origin xyz=-0.28302 0 0.048701 rpy=0 0 -1.5708 -> xyz=0 -0.28302 0.051876 rpy=0 0 0
- joint front_left_swivel_front_left_caster: origin xyz=-0.04445 0 -0.071438 rpy=0 0 0 -> xyz=-0.04445 0 -0.0714375 rpy=0 0 0

Commit message: fixed rviz lasers/mapping problem (wheel rpy)

File: urdf/coach_butler_robot.urdf (robot description, URDF)
Before this commit: robot coach_butler_robot, 12 links, 11 joints
Links:
- added link front_camera, mass 0.1; collision box size=0.05 0.05 0.05; visual box size=0.05 0.05 0.05
- added link rear_laser, mass 0.36783; collision mesh filename=package://butler_description/meshes/rear_laser.STL; visual mesh filename=package://butler_description/meshes/rear_laser.STL
Joints:
- added joint base_link_front_camera: type fixed, parent base_link, child front_camera, origin xyz=0.35239 0 1.32 rpy=0 0 0, axis 0 1 0
- added joint base_link_rear_laser: type revolute, parent base_link, child rear_laser, origin xyz=-0.38239 0 0.15967 rpy=0 0 3.14, axis 0 0 -1, limit lower=0 upper=0 effort=0 velocity=0
